Commit message: .

File: src/mobot_pkg/urdf/include/_body.urdf.xacro (robot description, xacro)
@@ -12,8 +12,8 @@
             </visual>
             <collision>
-                <origin rpy="0.0 0.0 0.0" xyz="0 0 0895"/>
+                <origin rpy="0.0 0.0 0.0" xyz="0 0 0405"/>
                 <geometry>
-                    <!-- <mesh filename="package://mobot_pkg/meshes/body.dae"/> -->
-                    <box size=".26 .15 .1"/>
+                    <!-- <mesh filename="package://mobot_pkg/meshes/Omobot_Version2_Body.dae"/> -->
+                    <box size=".288 .288 .150"/>
                     <!-- <mesh filename="${mesh}"/> -->
                 </geometry>
@@ -24,6 +24,6 @@
                 <inertia ixx="0.0060802336" ixy="0.0" ixz="0.0" iyy="0.0156763936" iyz="0.0" izz="0.02039184"/>
             </inertial> -->
-            <xacro:inertial_box mass="2" l=".26" w=".15" h=".002">
-                <origin rpy="0.0 0.0 0.0" xyz="0.0 0.0 0.002"/>
+            <xacro:inertial_box mass="3.4" l=".001" w=".001" h=".001">
+                <origin rpy="0.0 0.0 0.0" xyz="0.0 0.0 0.0405"/>
             </xacro:inertial_box>
         </link>

File: src/mobot_pkg/urdf/include/_camera.urdf.xacro (robot description, xacro)
@@ -19,6 +19,6 @@
                 </geometry>
             </collision>
-            <xacro:inertial_box mass=".03" l=".015" w=".015" h=".015">
-                <origin xyz="0 0 0.0065" rpy="0 0 0"/>
+            <xacro:inertial_box mass=".001" l=".001" w=".001" h=".001">
+                <origin xyz="0 0 0.0" rpy="0 0 0"/>
             </xacro:inertial_box>
         </link>

File: src/mobot_pkg/urdf/include/_imu.urdf.xacro (robot description, xacro)
@@ -22,5 +22,5 @@
             <inertial>
                 <origin rpy="0 0 0" xyz="0.0 0.0 0.0"/>
-                <mass value="0.005"/>
+                <mass value="0.001"/>
                 <inertia ixx=".00001" ixy="0.0" ixz="0.0" iyy=".001" iyz="0.0" izz=".00001"/>
             </inertial>

File: src/mobot_pkg/urdf/include/_lidar.urdf.xacro (robot description, xacro)
@@ -18,5 +18,5 @@
                 </geometry>
             </collision>
-            <xacro:inertial_cylinder mass=".03" rad=".015" hgt=".02">
+            <xacro:inertial_cylinder mass=".001" rad=".001" hgt=".001">
                 <origin xyz="-0 0 0" rpy="0 0 0"/>
             </xacro:inertial_cylinder>

File: src/mobot_pkg/urdf/omobot.urdf.xacro (robot description, xacro)
@@ -12,19 +12,19 @@
     <xacro:property name="wheel_length" value=".032"/>
     <!-- <xacro:property name="wheel_rad" value=".0395"/> -->
-    <xacro:body name_="base" parent_="base_footprint" x_="0.0" y_="0.0" z_="0" mat_="GRN" mesh="package://mobot_pkg/meshes/body_full.dae"/>
+    <xacro:body name_="base" parent_="base_footprint" x_="0.0" y_="0.0" z_="0" mat_="GRN" mesh="package://mobot_pkg/meshes/OmobotVersion2.dae"/>
     <gazebo reference="base_link">
         <material>Gazebo/Gray</material>
     </gazebo>
-    <xacro:fixed_components name_="jetson" parent_="base_link" mass_=".01" x_="0.01" y_="0" z_="0.126" l_="0.108" w_="0.102" h_="0.05" mat_="GRY"/>
-    <xacro:fixed_components name_="battery" parent_="base_link" mass_=".01" x_="0.0" y_="0.0" z_="0.0165" l_="0.05" w_="0.2" h_="0.03" mat_="GRY"/>
-    <xacro:lidar id_="1" parent_="base_link" x_="0.108" y_="0.0" z_="0.140" mat_="RED"/>
-    <xacro:imu id_="1" parent_="base_link" x_="0" y_="0.0" z_="0.095" mat_="RED"/>
-    <xacro:stereo_camera id_="1" parent_="base_link" x_="0.108" y_="0.0" z_="0.149" mat_="BLU"/>
-    <gazebo reference="jetson_link">
+    <!-- <xacro:fixed_components name_="jetson" parent_="base_link" mass_=".01" x_="0.01" y_="0" z_="0.126" l_="0.108" w_="0.102" h_="0.05" mat_="GRY"/>
+    <xacro:fixed_components name_="battery" parent_="base_link" mass_=".01" x_="0.0" y_="0.0" z_="0.0165" l_="0.05" w_="0.2" h_="0.03" mat_="GRY"/> -->
+    <xacro:lidar id_="1" parent_="base_link" x_="0.0975" y_="0.0" z_="0.1265" mat_="RED"/>
+    <xacro:imu id_="1" parent_="base_link" x_="0.013" y_="0.00" z_="0.0435" mat_="GRY"/>
+    <xacro:stereo_camera id_="1" parent_="base_link" x_="0.1325" y_="0.0" z_="0.069" mat_="BLU"/>
+    <!-- <gazebo reference="jetson_link">
         <material>Gazebo/Black</material>
     </gazebo>
     <gazebo reference="battery_link">
         <material>Gazebo/Black</material>
-    </gazebo>
+    </gazebo> -->
     <gazebo reference="lidar1_link">
         <material>Gazebo/Blue</material>
